File: 1 led blinking with 555ne.kicad_sch (KiCad schematic)
At the start: 6 parts

Commit message: Add files via upload
Connections:
- net at C2.1, R2.2: now also U?.2 (TR), U?.6 (THR)
Changed lines of the file:
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@@
   (junction (at 113.03 152.4) (diameter 0) (color 0 0 0 0)
+  )
+  (junction (at 143.51 102.87) (diameter 0) (color 0 0 0 0)
   )
   (junction (at 50.8 25.4) (diameter 0) (color 0 0 0 0)
@@
   )
   (junction (at 97.79 25.4) (diameter 0) (color 0 0 0 0)
+  )
+  (junction (at 50.8 132.08) (diameter 0) (color 0 0 0 0)
   )
   (junction (at 50.8 115.57) (diameter 0) (color 0 0 0 0)
@@
     (stroke (width 0) (type default) (color 0 0 0 0))
   )
+  (wire (pts (xy 143.51 102.87) (xy 143.51 132.08))
+    (stroke (width 0) (type default) (color 0 0 0 0))
+  )
   (wire (pts (xy 177.8 86.36) (xy 189.23 86.36))
     (stroke (width 0) (type default) (color 0 0 0 0))
@@
     (stroke (width 0) (type default) (color 0 0 0 0))
   )
+  (wire (pts (xy 143.51 132.08) (xy 50.8 132.08))
+    (stroke (width 0) (type default) (color 0 0 0 0))
+  )
   (wire (pts (xy 254 50.8) (xy 177.8 50.8))
     (stroke (width 0) (type default) (color 0 0 0 0))
@@
     (stroke (width 0) (type default) (color 0 0 0 0))
   )
+  (wire (pts (xy 50.8 132.08) (xy 50.8 134.62))
+    (stroke (width 0) (type default) (color 0 0 0 0))
+  )
   (wire (pts (xy 152.4 81.28) (xy 114.3 81.28))
     (stroke (width 0) (type default) (color 0 0 0 0))
   )
   (wire (pts (xy 50.8 115.57) (xy 205.74 115.57))
+    (stroke (width 0) (type default) (color 0 0 0 0))
+  )
+  (wire (pts (xy 50.8 124.46) (xy 50.8 132.08))
     (stroke (width 0) (type default) (color 0 0 0 0))
   )
@@
     (stroke (width 0) (type default) (color 0 0 0 0))
   )
-  (wire (pts (xy 50.8 124.46) (xy 50.8 134.62))
-    (stroke (width 0) (type default) (color 0 0 0 0))
-  )
